File: V1/esp-poe-backup.kicad_sch (KiCad schematic)
At the start: 48 parts, among them J1 USB_C_Receptacle_USB2.0, J2 RJ45 JACK, J3 PT1000 RTD, Q1 UMH3N, Q2 WPM2015-3/TR, Q3 LMUN2211LT1G, SW1 RESET, U4 CH340C, U5 ESP32-WROOM-32E-N4, U6 LAN8710A, U8 MAX31865xTP

Commit message: A lot of stuff
Parts:
- removed C27, C29: 100nF/50V, Tales:C_0402_1005Metric, symbol Device:C_Small
- removed C28: 10nF/50V, Tales:C_0402_1005Metric, symbol Device:C_Small
- removed J3: PT1000 RTD, Tales:TerminalBlock_Dibo_DB141R-2.54-2P_1x02_P2.54mm_Horizontal, symbol Connector_Generic:Conn_01x02
- removed R25: 4,02k/100mW, Tales:R_0603_1608Metric, symbol Device:R_US
- removed U8: MAX31865xTP, Tales:TQFN-20-1EP_5x5mm_P0.65mm_EP3.25x3.25mm_ThermalVias, symbol Sensor_Temperature:MAX31865xTP
- added C10, C11, C8: 100nF/50V, Tales:C_0402_1005Metric, symbol Device:C_Small
- added C9: 10nF/50V, Tales:C_0402_1005Metric, symbol Device:C_Small
- added J2: PT1000 RTD, Tales:TerminalBlock_Dibo_DB142R-5.08-2P_1x02_P5.08mm_Horizontal, symbol Connector_Generic:Conn_01x02
- added R6, R7: 2k2/62,5mW, Tales:R_0402_1005Metric, symbol Device:R_US
- added R8: 4,02k/100mW, Tales:R_0603_1608Metric, symbol Device:R_US
- added U2: MAX31865xTP, Package_DFN_QFN:TQFN-20-1EP_5x5mm_P0.65mm_EP3.25x3.25mm, symbol Sensor_Temperature:MAX31865xTP
- added U4: AHT20, Tales:DFN-6-3x3mm_P1mm, symbol Tales:AHT20
- U3: renamed from U5; Package ESP32-WROOM -> ESP32-WROOM-U
- renumbered C24 to C1, C15 to C12, C22 to C13, C23 to C14, C16 to C15, C17 to C16, C18 to C17, C19 to C18, C20 to C19, C10 to C2, C21 to C20, C25 to C3, C11 to C4, C12 to C5, C13 to C6, C14 to C7, D6 to D1, J2 to J3, L3 to L1, Q2 to Q1, Q3 to Q2, Q1 to Q3, R23 to R1, R18 to R10, R19 to R11, R21 to R12, R22 to R13, R20 to R14, R24 to R2, R14 to R3, R15 to R4, R16 to R5, R17 to R9, U4 to U1, U6 to U5
Connections:
- net +3.3V: now also C10.1, C11.1, C8.1, R6.1, R7.1, U2.19 (DVDD), U2.20 (VDD), U4.2 (VDD)
- net GND: now also C10.2, C11.2, C8.2, U2.10 (GND), U2.15 (DGND), U2.16 (GND), U2.21 (GND), U2.6 (FORCE2), U4.5 (GND)
- net SPI_CLK: now also U2.12 (SCLK)
- net SPI_CS: now also U2.13 (~{CS})
- net SPI_MISO: now also U2.14 (SDO)
- net SPI_MOSI: now also U2.11 (SDI)
- net I2C_SCL: now reaches U3.8 (IO32)
- net I2C_SCL: now also R6.2, U4.3 (SCL)
- net I2C_SDA: now reaches U3.9 (IO33)
- net I2C_SDA: now also R7.2, U4.4 (SDA)
- new net: C9.1, J2.1 (Pin_1), U2.5 (FORCE+), U2.7 (RTDIN+)
- new net: C9.2, J2.2 (Pin_2), U2.8 (RTDIN-), U2.9 (FORCE-)
- new net: R8.1, U2.1 (BIAS), U2.2 (REFIN+)
- new net: R8.2, U2.3 (REFIN-), U2.4 (ISENSOR)
- no-connect marks 28 -> 26
Other:
- note added: "TEMP/HUMID ADDRESS 0x38"
