File: V1/esp-poe-therm-v1.kicad_pcb (KiCad board)
At the start: 2 copper layers, 80 x 44 mm, 80 parts, among them J1 USB_C_Receptacle_USB2.0, J2 RJ45 JACK, J3 Sensor Temperatura, J4 Sensor Temperatura, Q1 UMH3N, Q2 WPM2015-3/TR, Q3 LMUN2211LT1G, SW1 RESET, U1 TPS2376DDAR-H, U2 TX4138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

Commit message: Work in progress
Parts:
- moved C26 19.3 mm to (146.0, 92.5)
- moved J4 19.3 mm to (149.0, 79.5)
- moved U7 19.3 mm to (146.0, 90.0)
- moved R1 0.50 mm to (124.5, 106.5)
Routing:
- net +3.3V: track 114.2 -> 122.9 mm, vias 5 -> 6
- net Net-(U1-UVLO): track 10.6 -> 9.28 mm
- net Net-(J2-RLED-): track 42.7 -> 43.2 mm
Other:
- board size 80 x 44 mm -> 76.5 x 44 mm
